File: ShildGSM.kicad_pcb (KiCad board)
At the start: 2 copper layers, 68.6 x 53.3 mm, 35 parts, among them P1 Power, P10 CONN_01X05, P14 CONN_01X07, P15 CONN_1, P16 CONN_1, P2 Analog, P3 Digital, P4 Digital, P5 CONN_1, P6 CONN_1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

Commit message: corectii
corectii in schema
Parts:
- added P11: CONN_01X02, Sockets_MOLEX_KK-System:Socket_MOLEX-KK-RM2-54mm_Lock_2pin_straight, F.Cu at (174.0, 110.3)
- added P12: CONN_01X02, Sockets_MOLEX_KK-System:Socket_MOLEX-KK-RM2-54mm_Lock_2pin_straight, F.Cu at (174.0, 104.8)
- added P13: CONN_01X02, Sockets_MOLEX_KK-System:Socket_MOLEX-KK-RM2-54mm_Lock_2pin_straight, F.Cu at (174.0, 99.4)
- P10: value CONN_01X05 -> CONN_01X02; footprint Terminal_Blocks:TerminalBlock_Pheonix_PT-3.5mm_5pol -> Sockets_MOLEX_KK-System:Socket_MOLEX-KK-RM2-54mm_Lock_2pin_straight
- P7: value CONN_1 -> CONN_01X02; footprint Socket_Arduino_Uno:Arduino_1pin -> Sockets_MOLEX_KK-System:Socket_MOLEX-KK-RM2-54mm_Lock_2pin_straight
- P9: value CONN_01X05 -> CONN_01X02; footprint Terminal_Blocks:TerminalBlock_Pheonix_PT-3.5mm_4pol -> Sockets_MOLEX_KK-System:Socket_MOLEX-KK-RM2-54mm_Lock_2pin_straight
- moved P7 60.2 mm to (117.7, 80.1), turned to 90 degrees
- moved P10 58.2 mm to (117.7, 97.1)
- moved P16 33.0 mm to (166.0, 80.4)
- moved C4 24.7 mm to (115.5, 92.9), turned to 0 degrees
- moved C6 24.6 mm to (115.7, 101.4), turned to 0 degrees
- moved C3 24.0 mm to (115.5, 84.4), turned to 0 degrees
- moved P8 15.2 mm to (177.0, 90.8)
- moved JP3 11.8 mm to (117.0, 75.1)
- moved P9 8.27 mm to (117.7, 88.6), turned to 90 degrees
- moved R4 6.71 mm to (171.0, 114.6)
- moved R5 6.13 mm to (127.0, 85.6), turned to 180 degrees
- moved R7 5.36 mm to (127.0, 92.9), turned to 180 degrees
- moved R1 5.22 mm to (126.7, 82.4)
- moved R8 4.47 mm to (127.7, 98.9), turned to 180 degrees
- moved R12 4.20 mm to (126.9, 79.6)
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Connections:
- C3 pad 2: /11(**/MOSI) -> Net-(C3-Pad2)
- C4 pad 2: /10(**/SS) -> Net-(C4-Pad2)
- C6 pad 2: /9(**) -> Net-(C6-Pad2)
- P10 pad 1: /A3 -> Net-(C6-Pad2)
- P10 pad 2: /A2 -> GND
- P7 pad 1: (no net) -> Net-(C3-Pad2)
- P9 pad 1: GND -> Net-(C4-Pad2)
- P9 pad 2: +5V -> GND
- R1 pad 2: Net-(P9-Pad3) -> Net-(C3-Pad2)
- R2 pad 2: Net-(P9-Pad4) -> Net-(C4-Pad2)
- R3 pad 2: (no net) -> Net-(C6-Pad2)
- R4 pad 2: Net-(P10-Pad3) -> Net-(P13-Pad2)
- R5 pad 2: /11(**/MOSI) -> Net-(C3-Pad2)
- R7 pad 2: /10(**/SS) -> Net-(C4-Pad2)
- R8 pad 2: /9(**) -> Net-(C6-Pad2)
Routing:
- net Net-(P10-Pad3): track 23.7 -> 0.00 mm
- net Net-(P13-Pad2): track 0.00 -> 17.3 mm
- net +5V: track 166.4 -> 180.5 mm
- net GND: track 293.0 -> 306.9 mm
- net /A5(SCL): track 8.93 -> 17.5 mm
- net /A4(SDA): track 9.09 -> 16.9 mm
- net Net-(P9-Pad4): track 6.63 -> 0.00 mm
- net Net-(P9-Pad3): track 6.55 -> 0.00 mm
- net /11(**/MOSI): track 27.6 -> 33.8 mm
- net Net-(C3-Pad2): track 0.00 -> 5.60 mm
- net /8: track 49.5 -> 46.9 mm
- net /10(**/SS): track 29.7 -> 31.8 mm
- net /A3: track 16.8 -> 14.9 mm
- net /A2: track 22.1 -> 23.6 mm
- net /9(**): track 38.8 -> 38.2 mm
- added copper zone on B.Cu, net Net-(C3-Pad2)
- added copper zone on B.Cu, net Net-(C4-Pad2)
- added copper zone on B.Cu, net Net-(C6-Pad2)

Commit message: LEDs
pus led err si led use
Parts:
- added D2: useLED, LEDs:LED-3MM, F.Cu at (137.9, 92.8)
- added D3: errLED, LEDs:LED-3MM, F.Cu at (137.9, 88.6)
- added R13: 1k, Discret:R3, F.Cu at (140.0, 82.2)
- added R6: 1k, Discret:R3, F.Cu at (143.4, 87.8)
- moved R11 1.30 mm to (134.6, 82.8)
Connections:
- P3 pad 5: (no net) -> /13(SCK)
- P3 pad 6: (no net) -> /12(MISO)
Routing:
- net /10(**/SS): track 31.8 -> 43.0 mm
- net /11(**/MOSI): track 33.8 -> 45.0 mm
- net /12(MISO): track 0.00 -> 9.17 mm
- net GND: track 306.9 -> 314.5 mm
- net /9(**): track 38.2 -> 42.2 mm
- net Net-(D2-Pad2): track 0.00 -> 3.49 mm
- net Net-(D3-Pad2): track 0.00 -> 2.75 mm
- net /8: track 46.9 -> 44.9 mm
- net /A4(SDA): track 16.9 -> 15.9 mm

Commit message: optimizat portare
Grupat R cu intrarile
Parts:
- moved R11 50.3 mm to (171.0, 117.5), turned to 0 degrees
- moved R10 9.21 mm to (164.6, 116.4), turned to 270 degrees
- moved D3 7.14 mm to (134.9, 82.1)
- moved D2 6.74 mm to (135.0, 86.7)
Routing:
- net GND: track 314.5 -> 306.0 mm
- net Net-(D2-Pad2): track 3.49 -> 9.75 mm
- net /A4(SDA): track 15.9 -> 10.4 mm
- net Net-(D3-Pad2): track 2.75 -> 6.40 mm
- net /13(SCK): track 0.00 -> 2.82 mm
- net /A2: track 23.6 -> 26.0 mm
- net /11(**/MOSI): track 45.0 -> 44.1 mm
- net /10(**/SS): track 43.0 -> 42.2 mm
